Commit message: Added a gripper and launch instructions.

File: ur_description/urdf/temoto_ur5_robot.urdf.xacro (robot description, xacro)
@@ -17,4 +17,5 @@
   <!-- NRG mods -->
   <!--          -->
+  <!-- Temoto frame -->
   <joint name="ee-temoto" type="fixed" >
     <origin xyz="0.22 0.0 0.0" rpy="-1.571 0 0"/>   <!-- place temoto_end_effector within the 2-finger gripper -->
@@ -23,3 +24,26 @@
   </joint>
   <link name="temoto_end_effector" />
+  <!-- Attach right gripper to arm -->
+  <joint name="ee-gripper" type="fixed">
+    <parent link= "ee_link" />
+    <child link = "2_finger_140_gripper_link" />
+    <origin xyz="0.0 0.04 0.1" rpy="1.5707 1.5707 0" />
+  </joint>
+  <link name="2_finger_140_gripper_link">
+    <visual>
+      <origin xyz="0.0 0.0 0.0" rpy="0.0 0.0 0.0" />
+      <geometry>
+        <mesh filename="package://ur_gazebo/meshes/2_finger_140_gripper.stl" scale="0.001 0.001 0.001"/>
+      </geometry>
+      <material name="black">
+        <color rgba="0.05 0.05 0.05 1"/>
+      </material>
+    </visual>
+    <collision>
+      <origin xyz="0.0 0.0 0.0" rpy="0.0 0.0 0.0" />
+      <geometry>
+        <mesh filename="package://ur_gazebo/meshes/2_finger_140_gripper.stl" scale="0.001 0.001 0.001"/>
+      </geometry>
+    </collision>
+  </link>
 </robot>

Commit message: Updating Temoto frame in URDF, adding floorplane link, and redoing the MoveIt setup assistant.

File: ur_description/urdf/temoto_ur5_robot.urdf.xacro (robot description, xacro)
@@ -17,11 +17,4 @@
   <!-- NRG mods -->
   <!--          -->
-  <!-- Temoto frame -->
-  <joint name="ee-temoto" type="fixed" >
-    <origin xyz="0.22 0.0 0.0" rpy="-1.571 0 0"/>   <!-- place temoto_end_effector within the 2-finger gripper -->
-    <parent link="ee_link" />  <!-- end-effector link for UR5 -->
-    <child link="temoto_end_effector" />
-  </joint>
-  <link name="temoto_end_effector" />
   <!-- Attach right gripper to arm -->
   <joint name="ee-gripper" type="fixed">

File: ur_description/urdf/ur5.urdf.xacro (robot description, xacro)
@@ -311,4 +311,36 @@
       <child link="${prefix}tool0"/>
     </joint>
+    <!-- NRG mods -->
+    <!-- Temoto frame -->
+    <joint name="ee-temoto" type="fixed" >
+      <origin xyz="0.22 0.0 0.0" rpy="-1.571 0 0"/>   <!-- place temoto_end_effector within the 2-finger gripper -->
+      <parent link="ee_link" />  <!-- end-effector link for UR5 -->
+      <child link="temoto_end_effector" />
+    </joint>
+    <link name="temoto_end_effector" />
+    <!-- add floorplane -->
+    <link name="floorplane_link">
+      <visual>
+        <origin xyz="0.0 0.0 0.0" rpy="0.0 0.0 0.0" />
+        <geometry>
+            <box size="1.0 1.0 0.05"/>
+        </geometry>
+        <material name="white">
+          <color rgba="1 1 1 0."/>
+        </material>
+      </visual>
+      <collision>
+        <origin xyz="0.0 0.0 0.0" rpy="0.0 0.0 0.0" />
+        <geometry>
+            <box size="1.0 1.0 0.05"/>
+        </geometry>
+        <material name="white"/>
+      </collision>
+    </link>
+    <joint name="floorplane_joint" type="fixed">
+      <parent link= "base_link" />
+      <child link = "floorplane_link" />
+      <origin xyz="0.0 0.0 0.0" rpy="0.0 0.0 0.0" />
+    </joint>
   </xacro:macro>
 </robot>

Commit message: Adding the Asus camera.

File: ur_description/urdf/temoto_ur5_robot.urdf.xacro (robot description, xacro)
@@ -12,5 +12,5 @@
     <parent link="world" />
     <child link = "base_link" />
-    <origin xyz="0.0 0.0 0.0" rpy="0.0 0.0 0.0" />
+    <origin xyz="0.0 -0.25 0.25" rpy="0.0 0.0 0.0" />
   </joint>
   <!--          -->
